File: Hardware Kicad/Venato.sch (KiCad schematic (older format))
At the start: 24 parts, among them U1 MCP6002-xMC, U2 MCP6002-xMC, U3 MCP6002-xMC, U4 MCP6002-xMC, U5 MCP6002-xMC, U6 MCP6002-xMC

Commit message: Added PCB
DRC ok, need to generate gerbers
Parts:
- removed C? (x6): 47pF, symbol Device:C
- removed R?: 1000, symbol Device:R
- removed U2, U3, U4, U5, U6, U? (x6): MCP6002-xMC, Package_DFN_QFN:DFN-8-1EP_3x2mm_P0.5mm_EP1.75x1.45mm, symbol Amplifier_Operational:MCP6002-xMC
- added C1, C4: 1u, Capacitor_THT:C_Rect_L7.0mm_W4.5mm_P5.00mm, symbol Device:C
- added C2: 10u, Capacitor_THT:CP_Radial_D4.0mm_P2.00mm, symbol Device:C
- added C3: 0.1u, Capacitor_THT:C_Rect_L7.0mm_W2.5mm_P5.00mm, symbol Device:C
- added J1, J2, J3, J4, J5, J6: Conn_01x02_Male, Connector_PinHeader_2.54mm:PinHeader_1x02_P2.54mm_Vertical, symbol Connector:Conn_01x02_Male
- added J7: Conn_01x05_Male, Connector_PinHeader_2.54mm:PinHeader_1x05_P2.54mm_Vertical, symbol Connector:Conn_01x05_Male
- added R4: 270, Resistor_THT:R_Axial_DIN0204_L3.6mm_D1.6mm_P7.62mm_Horizontal, symbol Device:R
- added R5: 180, Resistor_THT:R_Axial_DIN0204_L3.6mm_D1.6mm_P7.62mm_Horizontal, symbol Device:R
- added R6: 42k, Resistor_THT:R_Axial_DIN0204_L3.6mm_D1.6mm_P7.62mm_Horizontal, symbol Device:R
- added R7: 9k, Resistor_THT:R_Axial_DIN0204_L3.6mm_D1.6mm_P7.62mm_Horizontal, symbol Device:R
- added U1: LM317_TO-220, Package_TO_SOT_THT:TO-220-3_Vertical, symbol Regulator_Linear:LM317_TO-220
- added unit 2 of U2
- added unit 3 of U2
- added U3, U4: MCP6002-xP, Package_DIP:DIP-8_W7.62mm, symbol Amplifier_Operational:MCP6002-xP
- R1, R2, R3, R9: renamed from R?; value 1000 -> 1.5k; footprint (none) -> Resistor_THT:R_Axial_DIN0204_L3.6mm_D1.6mm_P7.62mm_Horizontal
- R8: renamed from R?; value R -> 1.5k; footprint (none) -> Resistor_THT:R_Axial_DIN0204_L3.6mm_D1.6mm_P7.62mm_Horizontal
- U2: renamed from U1; value MCP6002-xMC -> MCP6002-xP; footprint Package_DFN_QFN:DFN-8-1EP_3x2mm_P0.5mm_EP1.75x1.45mm -> Package_DIP:DIP-8_W7.62mm; symbol Amplifier_Operational:MCP6002-xMC -> Amplifier_Operational:MCP6002-xP
Connections:
- net SENSE1: now reaches R1.1, U2.1
- net SENSE1: now also J7.2 (Pin_2)
- net at R1.2, U2.2 (-): now also J1.1 (Pin_1)
- net SENSE2: now reaches R2.1
- net SENSE2: now also J7.1 (Pin_1), U3.1
- net at R2.2: now also J2.1 (Pin_1), U3.2 (-)
- net SENSE4: now reaches R3.1
- net SENSE4: now also J7.3 (Pin_3), U4.1
- net at R3.2: now also J3.1 (Pin_1), U4.2 (-)
- net at R9.2: now also J5.1 (Pin_1), U4.6 (-)
- net SENSE3: now reaches R9.1
- net SENSE3: now also J7.5 (Pin_5), U4.7
- net at R8.2: now also J4.1 (Pin_1), U2.6 (-)
- net SENSE5: now reaches R8.1
- net SENSE5: now also J7.4 (Pin_4), U2.7
- net 0 renamed VGND
- net VGND: now also U2.5 (+), U3.3 (+), U3.6 (-), U3.7, U4.3 (+), U4.5 (+)
- new net: R6.2, R7.1, U3.5 (+)
- new net: R4.2, R5.1, U1.1 (ADJ)
- new net +3.3VA: C2.1, C3.1, C4.1, R4.1, R6.1, U1.2 (VO), U2.8 (V+), U3.8 (V+), U4.8 (V+)
- new net +5V: C1.1, J6.1 (Pin_1), U1.3 (VI)
- new net GND: C1.2, C2.2, C3.2, C4.2, J1.2 (Pin_2), J2.2 (Pin_2), J3.2 (Pin_2), J4.2 (Pin_2), J5.2 (Pin_2), J6.2 (Pin_2), R5.2, R7.2, U2.4 (V-), U3.4 (V-), U4.4 (V-)
Other:
- moved on the sheet: R1, R2, R3, R8, R9, U2A
