File: Hardware v2/Venato.sch (KiCad schematic (older format))
At the start: 24 parts, among them J1 Conn_01x02_Male, J2 Conn_01x02_Male, J3 Conn_01x02_Male, J4 Conn_01x02_Male, J5 Conn_01x02_Male, J6 Conn_01x15_Female, J7 Conn_01x15_Female, U1 LM317_TO-220, U2 MCP6002-xP, U3 MCP6002-xP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

Commit message: v2 pcb done
Parts:
- added J8: Conn_01x02_Male, Connector_JST:JST_PH_B2B-PH-SM4-TB_1x02-1MP_P2.00mm_Vertical, symbol Connector:Conn_01x02_Male
- U1: footprint Package_TO_SOT_THT:TO-220-3_Vertical -> Package_TO_SOT_SMD:SOT-223
Connections:
- net GND: now also J8.2 (Pin_2)
- net VIN: now also J8.1 (Pin_1)
Changed lines of the file:
@@
 F 0 "U1" H 1650 1492 50  0000 C CNN
 F 1 "LM317_TO-220" H 1650 1401 50  0000 C CNN
-F 2 "Package_TO_SOT_THT:TO-220-3_Vertical" H 1650 1500 50  0001 C CIN
+F 2 "Package_TO_SOT_SMD:SOT-223" H 1650 1500 50  0001 C CIN
 F 3 "http://www.ti.com/lit/ds/symlink/lm317.pdf" H 1650 1250 50  0001 C CNN
 	1    1650 1250
@@
 Wire Wire Line
 	6100 5200 6250 5200
+$Comp
+L Connector:Conn_01x02_Male J8
+U 1 1 61E5B5DD
+P 6450 2850
+F 0 "J8" H 6558 3031 50  0000 C CNN
+F 1 "Conn_01x02_Male" H 6558 2940 50  0000 C CNN
+F 2 "Connector_JST:JST_PH_B2B-PH-SM4-TB_1x02-1MP_P2.00mm_Vertical" H 6450 2850 50  0001 C CNN
+F 3 "~" H 6450 2850 50  0001 C CNN
+	1    6450 2850
+	1    0    0    -1
+$EndComp
+Text GLabel 6750 2850 2    50   Input ~ 0
+VIN
+$Comp
+L power:GND #PWR0101
+U 1 1 61E67FF5
+P 6750 2950
+F 0 "#PWR0101" H 6750 2700 50  0001 C CNN
+F 1 "GND" H 6755 2777 50  0000 C CNN
+F 2 "" H 6750 2950 50  0001 C CNN
+F 3 "" H 6750 2950 50  0001 C CNN
+	1    6750 2950
+	1    0    0    -1
+$EndComp
+Wire Wire Line
+	6750 2950 6650 2950
+Wire Wire Line
+	6750 2850 6650 2850
 $EndSCHEMATC
